File: pcb/macro_keypad_pcb/macro_keypad_pcb.kicad_sch (KiCad schematic)
At the start: 13 parts, among them SW1 CHERRY_MX, SW2 CHERRY_MX, SW3 CHERRY_MX, SW4 CHERRY_MX, SW5 TL3305A, U1 Pico

Commit message: add example PCB layout
Parts:
- removed TP1: TestPoint, symbol Connector:TestPoint
- DISP1: footprint (none) -> Connector_PinHeader_2.54mm:PinHeader_1x04_P2.54mm_Vertical_SMD_Pin1Left
- SW1, SW2, SW3, SW4: symbol Switch:SW_MEC_5G -> Switch:SW_Push
- SW5: value TL3305A -> EQVP7C; footprint Button_Switch_SMD:SW_SPST_TL3305A -> macro_keypad:SW_SPST_EVQP7C; symbol Switch:SW_MEC_5E -> Switch:SW_Push
- U1: footprint RPi_Pico:RPi_Pico_SMD_TH -> MCU_RaspberryPi_and_Boards:RPi_Pico_SMD_TH
Connections:
- net +5V: now also SW1.2, SW2.2, SW3.2, SW4.2, SW5.2; no longer SW1.3 (B), SW1.4 (B), SW2.3 (B), SW2.4 (B), SW3.3 (B), SW3.4 (B), SW4.3 (B), SW4.4 (B), SW5.3 (K), SW5.4 (A)
- net switch_1: no longer SW1.2 (A)
- net switch_2: no longer SW2.2 (A)
- net switch_3: no longer SW3.2 (A)
- net switch_4: no longer SW4.2 (A)
- net switch_config: now also U1.12 (GPIO9); no longer SW5.2, U1.19 (GPIO14)
